File: hardware/gpib.kicad_sch (KiCad schematic)
At the start: 24 parts, among them J1 112-024-113R001, U3 SN75160BDW, U4 SN75161BDW

Commit message: hardware: 4-layer board, placement on both sides, J1 dimensioned
Takes the PCB from bare footprints to a fully placed 4-layer board. No
copper is routed yet and no zones are poured.

Stackup and outline
  Two inner copper layers added: In1.Cu intended as a solid ground plane
  directly beneath the component side, In2.Cu for power distribution. The
  board stays 62 x 68 mm. It is deliberately NOT grown: depth adds mass and
  lengthens the moment arm from the RJ45 cable back to the GPIB connector,
  and the mechanical load path is the connector's two M3 jackscrews on
  46.8 mm centres rather than its 24 signal contacts.

Placement
  All 90 footprints placed: 19 on F.Cu, 71 on B.Cu. Assembly is by hand, so
  back-side passives cost nothing and the 3D-printed enclosure accommodates
  them. Each decoupling capacitor sits on B.Cu directly beneath its IC's
  supply pin, so the connection is a through-via rather than a trace - the
  tightest supply loop available, and it costs no front-side area. That is
  what let the board stay 62 x 68 at ~35% front-side courtyard utilisation
  instead of the 68.7% a single-sided layout needed.

  Verified: zero courtyard overlaps; crystal load caps 0.00-4.00 mm from
  their crystals; C_U3a1 and C_U4a1 at 0.00 mm from their transceivers.

  Done with KiCad's own Flip() transform via the pcbnew Python API, one
  atomic pass, so pads, silkscreen, courtyards and 3D model offsets all
  moved correctly. auto_place_from_schematic was tried and rejected: it
  scored 15 -> 0, planned two parts to identical coordinates and put one
  off-board.

J1 GPIB connector
  Rotated 180 so the pad rows sit at the front edge and the shroud
  overhangs off-board, instead of the body consuming 24 mm of board depth.
  Set back so the two M3 mounting holes are 10.70 mm from the front edge
  per the mechanical drawing; hole span measures 46.80 mm, matching the
  datasheet. This costs 7.84 mm of board depth versus the earlier position
  and reduces the overhang to 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
Parts:
- C_SH1, C_U3a1, C_U3b1, C_U4a1, C_U4b1: footprint (none) -> Capacitor_SMD:C_0805_2012Metric
- R_ATN1, R_DC1, R_IFC1, R_PE1, R_REN1, R_SH1, R_SRQ1, R_TE1: footprint (none) -> Resistor_SMD:R_0805_2012Metric
- TP_ATN1, TP_DAV1, TP_DC1, TP_IFC1, TP_NDAC1, TP_NRFD1, TP_SRQ1, TP_TE1: footprint (none) -> TestPoint:TestPoint_Pad_D1.5mm
- U4: footprint adapter:SOIC-20_L13.0-W7.6-P1.27-LS10.3-BL -> Package_SO:SOIC-20W_7.5x12.8mm_P1.27mm
Changed lines of the file:
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@@
 			)
 		)
-		(property "Footprint" ""
+		(property "Footprint" "Capacitor_SMD:C_0805_2012Metric"
 			(at 200.66 137.16 0)
 			(hide yes)
@@
 			)
 		)
-		(property "Footprint" ""
+		(property "Footprint" "Resistor_SMD:R_0805_2012Metric"
 			(at 62.23 96.52 0)
 			(hide yes)
@@
 			)
 		)
-		(property "Footprint" ""
+		(property "Footprint" "TestPoint:TestPoint_Pad_D1.5mm"
 			(at 254 205.74 0)
 			(hide yes)
@@
 			)
 		)
-		(property "Footprint" ""
+		(property "Footprint" "Capacitor_SMD:C_0805_2012Metric"
 			(at 200.66 30.48 0)
 			(hide yes)
@@
 			)
 		)
-		(property "Footprint" ""
+		(property "Footprint" "Resistor_SMD:R_0805_2012Metric"
 			(at 43.18 215.9 0)
 			(hide yes)
@@
 			)
 		)
-		(property "Footprint" ""
+		(property "Footprint" "Capacitor_SMD:C_0805_2012Metric"
 			(at 215.9 137.16 0)
 			(hide yes)
@@
 			)
 		)
-		(property "Footprint" ""
+		(property "Footprint" "TestPoint:TestPoint_Pad_D1.5mm"
 			(at 228.6 205.74 0)
 			(hide yes)
@@
 			)
 		)
-		(property "Footprint" ""
+		(property "Footprint" "TestPoint:TestPoint_Pad_D1.5mm"
 			(at 62.23 86.36 0)
 			(hide yes)
@@
 			)
 		)
-		(property "Footprint" ""
+		(property "Footprint" "Capacitor_SMD:C_0805_2012Metric"
 			(at 215.9 30.48 0)
 			(hide yes)
@@
 			)
 		)
-		(property "Footprint" ""
+		(property "Footprint" "Resistor_SMD:R_0805_2012Metric"
 			(at 340.36 149.86 0)
 			(hide yes)
@@
 			)
 		)
-		(property "Footprint" ""
+		(property "Footprint" "TestPoint:TestPoint_Pad_D1.5mm"
 			(at 292.1 205.74 0)
 			(hide yes)
@@
 			)
 		)
-		(property "Footprint" ""
+		(property "Footprint" "Resistor_SMD:R_0805_2012Metric"
 			(at 175.26 30.48 0)
 			(hide yes)
@@
 			)
 		)
-		(property "Footprint" ""
+		(property "Footprint" "TestPoint:TestPoint_Pad_D1.5mm"
 			(at 279.4 205.74 0)
 			(hide yes)
@@
 			)
 		)
-		(property "Footprint" ""
+		(property "Footprint" "TestPoint:TestPoint_Pad_D1.5mm"
 			(at 77.47 86.36 0)
 			(hide yes)
@@
 			)
 		)
-		(property "Footprint" ""
+		(property "Footprint" "TestPoint:TestPoint_Pad_D1.5mm"
 			(at 266.7 205.74 0)
 			(hide yes)
@@
 			)
 		)
-		(property "Footprint" ""
+		(property "Footprint" "Resistor_SMD:R_0805_2012Metric"
 			(at 73.66 215.9 0)
 			(hide yes)
@@
 			)
 		)
-		(property "Footprint" ""
+		(property "Footprint" "Capacitor_SMD:C_0805_2012Metric"
 			(at 353.06 149.86 0)
 			(hide yes)
@@
 			)
 		)
-		(property "Footprint" ""
+		(property "Footprint" "Resistor_SMD:R_0805_2012Metric"
 			(at 77.47 96.52 0)
 			(hide yes)
@@
 			)
 		)
-		(property "Footprint" ""
+		(property "Footprint" "Resistor_SMD:R_0805_2012Metric"
 			(at 58.42 215.9 0)
 			(hide yes)
@@
 			)
 		)
-		(property "Footprint" ""
+		(property "Footprint" "Resistor_SMD:R_0805_2012Metric"
 			(at 88.9 215.9 0)
 			(hide yes)
@@
 			)
 		)
-		(property "Footprint" ""
+		(property "Footprint" "TestPoint:TestPoint_Pad_D1.5mm"
 			(at 241.3 205.74 0)
 			(hide yes)
@@
 			)
 		)
-		(property "Footprint" "adapter:SOIC-20_L13.0-W7.6-P1.27-LS10.3-BL"
+		(property "Footprint" "Package_SO:SOIC-20W_7.5x12.8mm_P1.27mm"
 			(at 139.7 175.26 0)
 			(hide yes)
