File: hardware/adapter.kicad_sch (KiCad schematic)
At the start: 0 parts

Commit message: hardware: USB-C alternate power source, J2 swapped to HanRun HR871150C
Implements the USB-C-as-alternative-power-source design (design-spec
§30.1): a 1x3 2.54mm header (J4) selects the system rail source via a
jumper rather than a diode-OR, since a Schottky drop would put +5V_SYS
below the SN75160B/161B's 4.75V minimum. Pin 1 = +5V_POE (M1's isolated
output), pin 2 = +5V_SYS (everything downstream), pin 3 = VBUS (from
J3's USB-C pads, already present with 5k1 CC pull-downs). R_G1/C_G1 stay
referenced to +5V_SYS along with Q1's source (R-HW-020): the gate
pull-up must track whichever rail the source actually sits on, or Q1
turns on with IOVDD absent whenever the other source is unpowered.

J2 (PoE RJ45) swapped from a generic MagJack footprint to the actual
ordered part, HanRun HR871150C (LCSC C19724786), correcting the PoE tap
pin numbers (J2.7-10, was J2.13-16) and the shield/ground pin scheme
against its real datasheet pinout.

Added docs/rp2354a-pinmap.md (RP2354A pin assignments) and
hardware/adapter.kicad_dru (project DRC rules). netlist-check.py's
bias-rail-discipline check extended to also flag +5V_SYS, matching the
new rail.
Parts:
- added H1, H2: MountingHole_Pad, MountingHole:MountingHole_3.2mm_M3_Pad, symbol Mechanical:MountingHole_Pad
Connections:
- new net GND: H1.1, H2.1
