File: hardware/mcu.kicad_sch (KiCad schematic)
At the start: 17 parts, among them J3 USB-C, U1 RP2354A, X1 12MHz

Commit message: hardware: 4-layer board, placement on both sides, J1 dimensioned
Takes the PCB from bare footprints to a fully placed 4-layer board. No
copper is routed yet and no zones are poured.

Stackup and outline
  Two inner copper layers added: In1.Cu intended as a solid ground plane
  directly beneath the component side, In2.Cu for power distribution. The
  board stays 62 x 68 mm. It is deliberately NOT grown: depth adds mass and
  lengthens the moment arm from the RJ45 cable back to the GPIB connector,
  and the mechanical load path is the connector's two M3 jackscrews on
  46.8 mm centres rather than its 24 signal contacts.

Placement
  All 90 footprints placed: 19 on F.Cu, 71 on B.Cu. Assembly is by hand, so
  back-side passives cost nothing and the 3D-printed enclosure accommodates
  them. Each decoupling capacitor sits on B.Cu directly beneath its IC's
  supply pin, so the connection is a through-via rather than a trace - the
  tightest supply loop available, and it costs no front-side area. That is
  what let the board stay 62 x 68 at ~35% front-side courtyard utilisation
  instead of the 68.7% a single-sided layout needed.

  Verified: zero courtyard overlaps; crystal load caps 0.00-4.00 mm from
  their crystals; C_U3a1 and C_U4a1 at 0.00 mm from their transceivers.

  Done with KiCad's own Flip() transform via the pcbnew Python API, one
  atomic pass, so pads, silkscreen, courtyards and 3D model offsets all
  moved correctly. auto_place_from_schematic was tried and rejected: it
  scored 15 -> 0, planned two parts to identical coordinates and put one
  off-board.

J1 GPIB connector
  Rotated 180 so the pad rows sit at the front edge and the shroud
  overhangs off-board, instead of the body consuming 24 mm of board depth.
  Set back so the two M3 mounting holes are 10.70 mm from the front edge
  per the mechanical drawing; hole span measures 46.80 mm, matching the
  datasheet. This costs 7.84 mm of board depth versus the earlier position
  and reduces the overhang to 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
Parts:
- C6, C7, C_X1a1, C_X1b1: footprint (none) -> Capacitor_SMD:C_0805_2012Metric
- L1: footprint (none) -> Inductor_SMD:L_0805_2012Metric
- LED1: footprint (none) -> LED_SMD:LED_0805_2012Metric
- R_CC1, R_CC2, R_CFG1, R_LED1, R_RUN1: footprint (none) -> Resistor_SMD:R_0805_2012Metric
- TP_GPIO221, TP_SWCLK1, TP_SWDIO1: footprint (none) -> TestPoint:TestPoint_Pad_D1.5mm
- X1: footprint (none) -> Crystal:Crystal_SMD_3225-4Pin_3.2x2.5mm
Changed lines of the file:
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@@
 			)
 		)
-		(property "Footprint" ""
+		(property "Footprint" "Capacitor_SMD:C_0805_2012Metric"
 			(at 91.44 124.46 0)
 			(hide yes)
@@
 			)
 		)
-		(property "Footprint" ""
+		(property "Footprint" "LED_SMD:LED_0805_2012Metric"
 			(at 260.35 175.26 0)
 			(hide yes)
@@
 			)
 		)
-		(property "Footprint" ""
+		(property "Footprint" "Capacitor_SMD:C_0805_2012Metric"
 			(at 106.68 124.46 0)
 			(hide yes)
@@
 			)
 		)
-		(property "Footprint" ""
+		(property "Footprint" "Capacitor_SMD:C_0805_2012Metric"
 			(at 121.92 151.13 0)
 			(hide yes)
@@
 			)
 		)
-		(property "Footprint" ""
+		(property "Footprint" "Inductor_SMD:L_0805_2012Metric"
 			(at 121.92 111.76 0)
 			(hide yes)
@@
 			)
 		)
-		(property "Footprint" ""
+		(property "Footprint" "Capacitor_SMD:C_0805_2012Metric"
 			(at 144.78 151.13 0)
 			(hide yes)
@@
 			)
 		)
-		(property "Footprint" ""
+		(property "Footprint" "Resistor_SMD:R_0805_2012Metric"
 			(at 320.04 74.93 0)
 			(hide yes)
@@
 			)
 		)
-		(property "Footprint" ""
+		(property "Footprint" "TestPoint:TestPoint_Pad_D1.5mm"
 			(at 139.7 124.46 0)
 			(hide yes)
@@
 			)
 		)
-		(property "Footprint" ""
+		(property "Footprint" "TestPoint:TestPoint_Pad_D1.5mm"
 			(at 241.3 167.64 0)
 			(hide yes)
@@
 			)
 		)
-		(property "Footprint" ""
+		(property "Footprint" "Resistor_SMD:R_0805_2012Metric"
 			(at 241.3 175.26 0)
 			(hide yes)
@@
 			)
 		)
-		(property "Footprint" ""
+		(property "Footprint" "Resistor_SMD:R_0805_2012Metric"
 			(at 146.05 68.58 0)
 			(hide yes)
@@
 			)
 		)
-		(property "Footprint" ""
+		(property "Footprint" "Resistor_SMD:R_0805_2012Metric"
 			(at 345.44 74.93 0)
 			(hide yes)
@@
 			)
 		)
-		(property "Footprint" ""
+		(property "Footprint" "Crystal:Crystal_SMD_3225-4Pin_3.2x2.5mm"
 			(at 133.35 146.05 0)
 			(hide yes)
@@
 			)
 		)
-		(property "Footprint" ""
+		(property "Footprint" "Resistor_SMD:R_0805_2012Metric"
 			(at 133.35 68.58 0)
 			(hide yes)
@@
 			)
 		)
-		(property "Footprint" ""
+		(property "Footprint" "TestPoint:TestPoint_Pad_D1.5mm"
 			(at 152.4 127 0)
 			(hide yes)

Commit message: hardware: USB-C alternate power source, J2 swapped to HanRun HR871150C
Implements the USB-C-as-alternative-power-source design (design-spec
§30.1): a 1x3 2.54mm header (J4) selects the system rail source via a
jumper rather than a diode-OR, since a Schottky drop would put +5V_SYS
below the SN75160B/161B's 4.75V minimum. Pin 1 = +5V_POE (M1's isolated
output), pin 2 = +5V_SYS (everything downstream), pin 3 = VBUS (from
J3's USB-C pads, already present with 5k1 CC pull-downs). R_G1/C_G1 stay
referenced to +5V_SYS along with Q1's source (R-HW-020): the gate
pull-up must track whichever rail the source actually sits on, or Q1
turns on with IOVDD absent whenever the other source is unpowered.

J2 (PoE RJ45) swapped from a generic MagJack footprint to the actual
ordered part, HanRun HR871150C (LCSC C19724786), correcting the PoE tap
pin numbers (J2.7-10, was J2.13-16) and the shield/ground pin scheme
against its real datasheet pinout.

Added docs/rp2354a-pinmap.md (RP2354A pin assignments) and
hardware/adapter.kicad_dru (project DRC rules). netlist-check.py's
bias-rail-discipline check extended to also flag +5V_SYS, matching the
new rail.
Connections:
- net VBUS: now reaches J3.A4B9 (VBUS)
- net VBUS: now also J3.B4A9 (VBUS)
- no-connect marks 13 -> 11
Changed lines of the file:
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@@
-	)
-	(no_connect
-		(at 96.52 50.8)
 	)
 	(no_connect
@@
 		(at 168.91 175.26)
 	)
-	(no_connect
-		(at 96.52 73.66)
+	(wire
+		(pts
+			(xy 96.52 50.8)
+			(xy 93.98 50.8)
+		)
+	)
+	(wire
+		(pts
+			(xy 96.52 73.66)
+			(xy 93.98 73.66)
+		)
 	)
 	(label "DVDD"
@@
 			)
 			(justify right bottom)
+		)
+	)
+	(global_label "VBUS"
+		(shape input)
+		(at 93.98 50.8 180)
+		(effects
+			(font
+				(size 1.27 1.27)
+			)
+			(justify right)
+		)
+	)
+	(global_label "VBUS"
+		(shape input)
+		(at 93.98 73.66 180)
+		(effects
+			(font
+				(size 1.27 1.27)
+			)
+			(justify right)
 		)
 	)
@@
 		(at 91.44 124.46 0)
 		(unit 1)
-		(body_style 1)
 		(exclude_from_sim no)
 		(in_bom yes)
 		(on_board yes)
-		(in_pos_files yes)
 		(dnp no)
 		(property "Reference" "C6"
@@
 			)
 		)
+		(body_style 1)
+		(in_pos_files yes)
 		(pin "1"
 		)
@@
 		(at 260.35 175.26 0)
 		(unit 1)
-		(body_style 1)
 		(exclude_from_sim no)
 		(in_bom yes)
 		(on_board yes)
-		(in_pos_files yes)
 		(dnp no)
 		(property "Reference" "LED1"
@@
 			)
 		)
+		(body_style 1)
+		(in_pos_files yes)
 		(pin "1"
 		)
@@
 		(at 106.68 124.46 0)
 		(unit 1)
-		(body_style 1)
 		(exclude_from_sim no)
 		(in_bom yes)
 		(on_board yes)
-		(in_pos_files yes)
 		(dnp no)
 		(property "Reference" "C7"
@@
 			)
 		)
+		(body_style 1)
+		(in_pos_files yes)
 		(pin "1"
 		)
@@
 		(at 121.92 151.13 0)
 		(unit 1)
-		(body_style 1)
 		(exclude_from_sim no)
 		(in_bom yes)
 		(on_board yes)
-		(in_pos_files yes)
 		(dnp no)
 		(property "Reference" "C_X1a1"
@@
 			)
 		)
+		(body_style 1)
+		(in_pos_files yes)
 		(pin "1"
 		)
@@
 		(at 121.92 111.76 0)
 		(unit 1)
-		(body_style 1)
 		(exclude_from_sim no)
 		(in_bom yes)
 		(on_board yes)
-		(in_pos_files yes)
 		(dnp no)
 		(property "Reference" "L1"
@@
 			)
 		)
+		(body_style 1)
+		(in_pos_files yes)
 		(pin "1"
 		)
@@
 		(at 144.78 151.13 0)
 		(unit 1)
-		(body_style 1)
 		(exclude_from_sim no)
 		(in_bom yes)
 		(on_board yes)
-		(in_pos_files yes)
 		(dnp no)
 		(property "Reference" "C_X1b1"
@@
 			)
 		)
+		(body_style 1)
+		(in_pos_files yes)
 		(pin "1"
 		)
@@
 		(at 168.91 160.02 180)
 		(unit 1)
-		(body_style 1)
 		(exclude_from_sim no)
 		(in_bom yes)
 		(on_board yes)
-		(in_pos_files yes)
 		(dnp no)
 		(property "Reference" "#PWR017"
@@
 			)
 		)
+		(body_style 1)
+		(in_pos_files yes)
 		(pin "1"
 		)
@@
 		(at 320.04 74.93 0)
 		(unit 1)
-		(body_style 1)
 		(exclude_from_sim no)
 		(in_bom yes)
 		(on_board yes)
-		(in_pos_files yes)
 		(dnp no)
 		(property "Reference" "R_RUN1"
@@
 			)
 		)
+		(body_style 1)
+		(in_pos_files yes)
 		(pin "1"
 		)
@@
 		(at 139.7 124.46 0)
 		(unit 1)
-		(body_style 1)
 		(exclude_from_sim no)
 		(in_bom yes)
 		(on_board yes)
-		(in_pos_files yes)
 		(dnp no)
 		(property "Reference" "TP_SWCLK1"
@@
 			)
 		)
+		(body_style 1)
+		(in_pos_files yes)
 		(pin "1"
 		)
@@
 		(at 102.87 62.23 0)
 		(unit 1)
-		(body_style 1)
 		(exclude_from_sim no)
 		(in_bom yes)
 		(on_board yes)
-		(in_pos_files yes)
 		(dnp no)
 		(property "Reference" "J3"
@@
 			)
 		)
+		(body_style 1)
+		(in_pos_files yes)
 		(pin "1"
 		)
@@
 		(at 241.3 167.64 0)
 		(unit 1)
-		(body_style 1)
 		(exclude_from_sim no)
 		(in_bom yes)
 		(on_board yes)
-		(in_pos_files yes)
 		(dnp no)
 		(property "Reference" "TP_GPIO221"
@@
 			)
 		)
+		(body_style 1)
+		(in_pos_files yes)
 		(pin "1"
 		)
@@
 		(at 241.3 175.26 0)
 		(unit 1)
-		(body_style 1)
 		(exclude_from_sim no)
 		(in_bom yes)
 		(on_board yes)
-		(in_pos_files yes)
 		(dnp no)
 		(property "Reference" "R_LED1"
@@
 			)
 		)
+		(body_style 1)
+		(in_pos_files yes)
 		(pin "1"
 		)
@@
 		(at 190.5 148.59 0)
 		(unit 1)
-		(body_style 1)
 		(exclude_from_sim no)
 		(in_bom yes)
 		(on_board yes)
-		(in_pos_files yes)
 		(dnp no)
 		(property "Reference" "U1"
@@
 			)
 		)
+		(body_style 1)
+		(in_pos_files yes)
 		(pin "35"
 		)
@@
 		(at 146.05 68.58 0)
 		(unit 1)
-		(body_style 1)
 		(exclude_from_sim no)
 		(in_bom yes)
 		(on_board yes)
-		(in_pos_files yes)
 		(dnp no)
 		(property "Reference" "R_CC2"
@@
 			)
 		)
+		(body_style 1)
+		(in_pos_files yes)
 		(pin "1"
 		)
@@
 		(at 345.44 74.93 0)
 		(unit 1)
-		(body_style 1)
 		(exclude_from_sim no)
 		(in_bom yes)
 		(on_board yes)
-		(in_pos_files yes)
 		(dnp no)
 		(property "Reference" "R_CFG1"
@@
 			)
 		)
+		(body_style 1)
+		(in_pos_files yes)
 		(pin "1"
 		)
@@
 		(at 133.35 146.05 0)
 		(unit 1)
-		(body_style 1)
 		(exclude_from_sim no)
 		(in_bom yes)
 		(on_board yes)
-		(in_pos_files yes)
 		(dnp no)
 		(property "Reference" "X1"
@@
 			)
 		)
+		(body_style 1)
+		(in_pos_files yes)
 		(pin "1"
 		)
@@
 		(at 186.69 208.28 0)
 		(unit 1)
-		(body_style 1)
 		(exclude_from_sim no)
 		(in_bom yes)
 		(on_board yes)
-		(in_pos_files yes)
 		(dnp no)
 		(property "Reference" "#PWR018"
@@
 			)
 		)
+		(body_style 1)
+		(in_pos_files yes)
 		(pin "1"
 		)
@@
 		(at 133.35 68.58 0)
 		(unit 1)
-		(body_style 1)
 		(exclude_from_sim no)
 		(in_bom yes)
 		(on_board yes)
-		(in_pos_files yes)
 		(dnp no)
 		(property "Reference" "R_CC1"
@@
 			)
 		)
+		(body_style 1)
+		(in_pos_files yes)
 		(pin "1"
 		)
@@
 		(at 152.4 127 0)
 		(unit 1)
-		(body_style 1)
 		(exclude_from_sim no)
 		(in_bom yes)
 		(on_board yes)
-		(in_pos_files yes)
 		(dnp no)
 		(property "Reference" "TP_SWDIO1"
@@
 			)
 		)
+		(body_style 1)
+		(in_pos_files yes)
 		(pin "1"
 		)
