File: hardware/power_gate.kicad_sch (KiCad schematic)
At the start: 14 parts, among them Q1 AO3401A, Q2 2N7002, U5 AP2114H-3.3TRG1, U6 TPS3839G33DBZR

Commit message: hardware: 4-layer board, placement on both sides, J1 dimensioned
Takes the PCB from bare footprints to a fully placed 4-layer board. No
copper is routed yet and no zones are poured.

Stackup and outline
  Two inner copper layers added: In1.Cu intended as a solid ground plane
  directly beneath the component side, In2.Cu for power distribution. The
  board stays 62 x 68 mm. It is deliberately NOT grown: depth adds mass and
  lengthens the moment arm from the RJ45 cable back to the GPIB connector,
  and the mechanical load path is the connector's two M3 jackscrews on
  46.8 mm centres rather than its 24 signal contacts.

Placement
  All 90 footprints placed: 19 on F.Cu, 71 on B.Cu. Assembly is by hand, so
  back-side passives cost nothing and the 3D-printed enclosure accommodates
  them. Each decoupling capacitor sits on B.Cu directly beneath its IC's
  supply pin, so the connection is a through-via rather than a trace - the
  tightest supply loop available, and it costs no front-side area. That is
  what let the board stay 62 x 68 at ~35% front-side courtyard utilisation
  instead of the 68.7% a single-sided layout needed.

  Verified: zero courtyard overlaps; crystal load caps 0.00-4.00 mm from
  their crystals; C_U3a1 and C_U4a1 at 0.00 mm from their transceivers.

  Done with KiCad's own Flip() transform via the pcbnew Python API, one
  atomic pass, so pads, silkscreen, courtyards and 3D model offsets all
  moved correctly. auto_place_from_schematic was tried and rejected: it
  scored 15 -> 0, planned two parts to identical coordinates and put one
  off-board.

J1 GPIB connector
  Rotated 180 so the pad rows sit at the front edge and the shroud
  overhangs off-board, instead of the body consuming 24 mm of board depth.
  Set back so the two M3 mounting holes are 10.70 mm from the front edge
  per the mechanical drawing; hole span measures 46.80 mm, matching the
  datasheet. This costs 7.84 mm of board depth versus the earlier position
  and reduces the overhang to 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
Parts:
- C_3V3, C_G1, C_LDOin1, C_LDOout1: footprint (none) -> Capacitor_SMD:C_0805_2012Metric
- C_BULK1: footprint (none) -> Capacitor_SMD:C_1206_3216Metric
- R_G1, R_G2: footprint (none) -> Resistor_SMD:R_0805_2012Metric
- TP_3V3, TP_5V1, TP_GND1: footprint (none) -> TestPoint:TestPoint_Pad_D1.5mm
Changed lines of the file:
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@@
 			)
 		)
-		(property "Footprint" ""
+		(property "Footprint" "Capacitor_SMD:C_0805_2012Metric"
 			(at 218.44 35.56 0)
 			(hide yes)
@@
 			)
 		)
-		(property "Footprint" ""
+		(property "Footprint" "Resistor_SMD:R_0805_2012Metric"
 			(at 170.18 74.93 0)
 			(hide yes)
@@
 			)
 		)
-		(property "Footprint" ""
+		(property "Footprint" "TestPoint:TestPoint_Pad_D1.5mm"
 			(at 132.08 38.1 0)
 			(hide yes)
@@
 			)
 		)
-		(property "Footprint" ""
+		(property "Footprint" "Capacitor_SMD:C_0805_2012Metric"
 			(at 119.38 54.61 0)
 			(hide yes)
@@
 			)
 		)
-		(property "Footprint" ""
+		(property "Footprint" "Capacitor_SMD:C_0805_2012Metric"
 			(at 105.41 54.61 0)
 			(hide yes)
@@
 			)
 		)
-		(property "Footprint" ""
+		(property "Footprint" "Capacitor_SMD:C_1206_3216Metric"
 			(at 44.45 54.61 0)
 			(hide yes)
@@
 			)
 		)
-		(property "Footprint" ""
+		(property "Footprint" "TestPoint:TestPoint_Pad_D1.5mm"
 			(at 69.85 21.59 0)
 			(hide yes)
@@
 			)
 		)
-		(property "Footprint" ""
+		(property "Footprint" "Capacitor_SMD:C_0805_2012Metric"
 			(at 59.69 54.61 0)
 			(hide yes)
@@
 			)
 		)
-		(property "Footprint" ""
+		(property "Footprint" "TestPoint:TestPoint_Pad_D1.5mm"
 			(at 105.41 73.66 0)
 			(hide yes)
@@
 			)
 		)
-		(property "Footprint" ""
+		(property "Footprint" "Resistor_SMD:R_0805_2012Metric"
 			(at 204.47 35.56 0)
 			(hide yes)

Commit message: hardware: USB-C alternate power source, J2 swapped to HanRun HR871150C
Implements the USB-C-as-alternative-power-source design (design-spec
§30.1): a 1x3 2.54mm header (J4) selects the system rail source via a
jumper rather than a diode-OR, since a Schottky drop would put +5V_SYS
below the SN75160B/161B's 4.75V minimum. Pin 1 = +5V_POE (M1's isolated
output), pin 2 = +5V_SYS (everything downstream), pin 3 = VBUS (from
J3's USB-C pads, already present with 5k1 CC pull-downs). R_G1/C_G1 stay
referenced to +5V_SYS along with Q1's source (R-HW-020): the gate
pull-up must track whichever rail the source actually sits on, or Q1
turns on with IOVDD absent whenever the other source is unpowered.

J2 (PoE RJ45) swapped from a generic MagJack footprint to the actual
ordered part, HanRun HR871150C (LCSC C19724786), correcting the PoE tap
pin numbers (J2.7-10, was J2.13-16) and the shield/ground pin scheme
against its real datasheet pinout.

Added docs/rp2354a-pinmap.md (RP2354A pin assignments) and
hardware/adapter.kicad_dru (project DRC rules). netlist-check.py's
bias-rail-discipline check extended to also flag +5V_SYS, matching the
new rail.
Parts:
- added J4: PWR_SEL, Connector_PinHeader_2.54mm:PinHeader_1x03_P2.54mm_Vertical, symbol Connector_Generic:Conn_01x03
Connections:
- net +5V_POE: now also J4.1 (Pin_1); no longer C_BULK1.1, C_G1.1, C_LDOin1.1, Q1.2 (S), R_G1.1, TP_5V1.1, U5.3 (VIN)
- new net +5V_SYS: C_BULK1.1, C_G1.1, C_LDOin1.1, J4.2 (Pin_2), Q1.2 (S), R_G1.1, TP_5V1.1, U5.3 (VIN)
- new net VBUS: J4.3 (Pin_3)
